File: hardware/precharge-outline/precharge.kicad_sch (KiCad schematic)
At the start: 16 parts

Commit message: Misc. changes to schematic, created PCB
The PCB was created just to begin modelling its size.
Parts:
- R?: value 1200 -> 680
- R?: value 3000 -> 4500
Changed lines of the file:
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@@
 (kicad_sch (version 20210621) (generator eeschema)
   (paper "A4")
-  (junction (at 194.31 140.97) (diameter 0) (color 0 0 0 0))
+  (junction (at 49.53 115.57) (diameter 0) (color 0 0 0 0))
+  (junction (at 45.72 57.15) (diameter 0) (color 0 0 0 0))
   (junction (at 35.56 168.91) (diameter 0) (color 0 0 0 0))
   (junction (at 106.68 59.69) (diameter 0) (color 0 0 0 0))
   (junction (at 191.77 59.69) (diameter 0) (color 0 0 0 0))
+  (junction (at 49.53 57.15) (diameter 0) (color 0 0 0 0))
   (junction (at 77.47 132.08) (diameter 0) (color 0 0 0 0))
-  (junction (at 49.53 115.57) (diameter 0) (color 0 0 0 0))
+  (junction (at 194.31 140.97) (diameter 0) (color 0 0 0 0))
   (junction (at 49.53 125.73) (diameter 0) (color 0 0 0 0))
-  (junction (at 45.72 57.15) (diameter 0) (color 0 0 0 0))
-  (junction (at 49.53 57.15) (diameter 0) (color 0 0 0 0))
   (no_connect (at 62.23 97.79))
   (wire (pts (xy 152.4 171.45) (xy 152.4 140.97))
@@
     (stroke (width 0) (type default) (color 0 0 0 0))
   )
+  (wire (pts (xy 62.23 87.63) (xy 57.15 87.63))
+    (stroke (width 0) (type default) (color 0 0 0 0))
+  )
+  (wire (pts (xy 57.15 87.63) (xy 57.15 105.41))
+    (stroke (width 0) (type default) (color 0 0 0 0))
+  )
   (wire (pts (xy 57.15 105.41) (xy 72.39 105.41))
     (stroke (width 0) (type default) (color 0 0 0 0))
@@
     (stroke (width 0) (type default) (color 0 0 0 0))
   )
-  (wire (pts (xy 62.23 87.63) (xy 57.15 87.63))
-    (stroke (width 0) (type default) (color 0 0 0 0))
-  )
-  (wire (pts (xy 57.15 87.63) (xy 57.15 105.41))
-    (stroke (width 0) (type default) (color 0 0 0 0))
-  )
   (wire (pts (xy 93.98 82.55) (xy 93.98 87.63))
     (stroke (width 0) (type default) (color 0 0 0 0))
@@
     (stroke (width 0) (type default) (color 0 0 0 0))
   )
+  (wire (pts (xy 194.31 140.97) (xy 241.3 140.97))
+    (stroke (width 1) (type default) (color 0 0 0 0))
+  )
   (wire (pts (xy 241.3 140.97) (xy 241.3 109.22))
     (stroke (width 1) (type default) (color 0 0 0 0))
   )
-  (wire (pts (xy 194.31 140.97) (xy 241.3 140.97))
-    (stroke (width 1) (type default) (color 0 0 0 0))
-  )
   (wire (pts (xy 81.28 21.59) (xy 81.28 24.13))
     (stroke (width 0) (type default) (color 0 0 0 0))
@@
     (stroke (width 0) (type default) (color 0 0 0 0))
   )
+  (wire (pts (xy 241.3 59.69) (xy 191.77 59.69))
+    (stroke (width 1) (type default) (color 0 0 0 0))
+  )
+  (wire (pts (xy 191.77 59.69) (xy 106.68 59.69))
+    (stroke (width 1) (type default) (color 0 0 0 0))
+  )
   (wire (pts (xy 241.3 101.6) (xy 241.3 59.69))
     (stroke (width 1) (type default) (color 0 0 0 0))
   )
-  (wire (pts (xy 191.77 59.69) (xy 106.68 59.69))
-    (stroke (width 1) (type default) (color 0 0 0 0))
-  )
-  (wire (pts (xy 241.3 59.69) (xy 191.77 59.69))
-    (stroke (width 1) (type default) (color 0 0 0 0))
-  )
   (wire (pts (xy 194.31 101.6) (xy 194.31 110.49))
     (stroke (width 0) (type default) (color 0 0 0 0))
@@
     (stroke (width 0) (type default) (color 0 0 0 0))
   )
+  (wire (pts (xy 85.09 118.11) (xy 148.59 118.11))
+    (stroke (width 0) (type default) (color 0 0 0 0))
+  )
   (wire (pts (xy 148.59 118.11) (xy 148.59 29.21))
     (stroke (width 0) (type default) (color 0 0 0 0))
   )
-  (wire (pts (xy 85.09 118.11) (xy 148.59 118.11))
-    (stroke (width 0) (type default) (color 0 0 0 0))
-  )
   (wire (pts (xy 148.59 29.21) (xy 218.44 29.21))
     (stroke (width 0) (type default) (color 0 0 0 0))
   )
+  (polyline (pts (xy 29.21 13.97) (xy 162.56 13.97))
+    (stroke (width 0) (type default) (color 0 0 0 0))
+  )
   (polyline (pts (xy 29.21 13.97) (xy 29.21 186.69))
     (stroke (width 0) (type default) (color 0 0 0 0))
@@
     (stroke (width 0) (type default) (color 0 0 0 0))
   )
-  (polyline (pts (xy 29.21 13.97) (xy 162.56 13.97))
-    (stroke (width 0) (type default) (color 0 0 0 0))
-  )
   (wire (pts (xy 49.53 57.15) (xy 49.53 100.33))
     (stroke (width 0) (type default) (color 0 0 0 0))
   )
+  (wire (pts (xy 93.98 97.79) (xy 93.98 102.87))
+    (stroke (width 0) (type default) (color 0 0 0 0))
+  )
   (wire (pts (xy 87.63 97.79) (xy 93.98 97.79))
     (stroke (width 0) (type default) (color 0 0 0 0))
   )
-  (wire (pts (xy 93.98 97.79) (xy 93.98 102.87))
-    (stroke (width 0) (type default) (color 0 0 0 0))
-  )
   (wire (pts (xy 49.53 115.57) (xy 49.53 116.84))
     (stroke (width 0) (type default) (color 0 0 0 0))
@@
     (stroke (width 0) (type default) (color 0 0 0 0))
   )
+  (wire (pts (xy 88.9 123.19) (xy 88.9 132.08))
+    (stroke (width 0) (type default) (color 0 0 0 0))
+  )
   (wire (pts (xy 88.9 132.08) (xy 77.47 132.08))
     (stroke (width 0) (type default) (color 0 0 0 0))
   )
-  (wire (pts (xy 88.9 123.19) (xy 88.9 132.08))
-    (stroke (width 0) (type default) (color 0 0 0 0))
-  )
   (wire (pts (xy 85.09 123.19) (xy 88.9 123.19))
     (stroke (width 0) (type default) (color 0 0 0 0))
@@
     (stroke (width 1) (type default) (color 0 0 0 0))
   )
+  (wire (pts (xy 99.06 36.83) (xy 106.68 36.83))
+    (stroke (width 0) (type default) (color 0 0 0 0))
+  )
   (wire (pts (xy 106.68 59.69) (xy 106.68 36.83))
     (stroke (width 0) (type default) (color 0 0 0 0))
   )
-  (wire (pts (xy 99.06 36.83) (xy 106.68 36.83))
-    (stroke (width 0) (type default) (color 0 0 0 0))
-  )
   (polyline (pts (xy 74.93 15.24) (xy 74.93 185.42))
     (stroke (width 0) (type default) (color 0 0 0 0))
@@
     (stroke (width 1) (type default) (color 0 0 0 0))
   )
+  (wire (pts (xy 35.56 57.15) (xy 45.72 57.15))
+    (stroke (width 1) (type default) (color 0 0 0 0))
+  )
+  (wire (pts (xy 45.72 57.15) (xy 49.53 57.15))
+    (stroke (width 1) (type default) (color 0 0 0 0))
+  )
+  (wire (pts (xy 35.56 93.98) (xy 35.56 57.15))
+    (stroke (width 1) (type default) (color 0 0 0 0))
+  )
   (wire (pts (xy 49.53 57.15) (xy 67.31 57.15))
-    (stroke (width 1) (type default) (color 0 0 0 0))
-  )
-  (wire (pts (xy 35.56 57.15) (xy 45.72 57.15))
-    (stroke (width 1) (type default) (color 0 0 0 0))
-  )
-  (wire (pts (xy 45.72 57.15) (xy 49.53 57.15))
-    (stroke (width 1) (type default) (color 0 0 0 0))
-  )
-  (wire (pts (xy 35.56 93.98) (xy 35.56 57.15))
     (stroke (width 1) (type default) (color 0 0 0 0))
   )
@@
     (in_bom yes) (on_board yes) (fields_autoplaced)
     (property "Reference" "R?" (id 0) (at 95.25 31.8475 90))
-    (property "Value" "1200" (id 1) (at 95.25 34.6226 90))
+    (property "Value" "680" (id 1) (at 95.25 34.6226 90))
     (property "Footprint" "" (id 2) (at 95.25 38.608 90)
       (effects (font (size 1.27 1.27)) hide)
@@
       (effects (font (size 1.27 1.27)) (justify left))
     )
-    (property "Value" "3000" (id 1) (at 196.088 116.1666 0)
+    (property "Value" "4500" (id 1) (at 196.088 116.1666 0)
       (effects (font (size 1.27 1.27)) (justify left))
     )
@@
     )
     (path "/48ae560b-46a8-4524-a114-9238cbbf797d"
-      (reference "R?") (unit 1) (value "1200") (footprint "")
+      (reference "R?") (unit 1) (value "680") (footprint "")
     )
     (path "/b4de5946-04c7-4df0-883b-43022546f9fc"
-      (reference "R?") (unit 1) (value "3000") (footprint "")
+      (reference "R?") (unit 1) (value "4500") (footprint "")
     )
     (path "/bf6c7fa0-d50c-4d12-9a1d-5261abd2ef28"
