File: hardware/precharge/indicator.kicad_sch (KiCad schematic)
At the start: 15 parts, among them Q9 XP262N7002TR-G, U6 OP777

Commit message: Latest precharge updates
Parts:
- removed D17: BZX84C12L, Package_TO_SOT_SMD:SOT-23, symbol Diode:BZX84Cxx
- removed D18: BZX84C6V2L, Package_TO_SOT_SMD:SOT-23, symbol Diode:BZX84Cxx
- added D17: MMSZ4699T1G, Diode_SMD:D_SOD-123, symbol Diode:1N630xA
- added D18: MMSZ4691T1G, Diode_SMD:D_SOD-123, symbol Diode:1N630xA
- J8: value (none) -> LED; footprint (none) -> footprints:Molex_Micro-Fit_3.0_43650-0200_1x02_P3.00mm_Horizontal
- Q8: value (none) -> FQD1N80TM; footprint (none) -> Package_TO_SOT_SMD:TO-252-2
Connections:
- net TS-: now also D17.2 (A2), D18.2 (A2)
- net at R71.1, U6.2 (-): now also D18.1 (A1)
- net at Q8.1 (G), R67.1: now also D17.1 (A1)
Other:
- note added: "For reference, some Farnell codes: FET: 2453434 12V Zener: 1651593 6.2V Zener: 2463561"
- note removed: "For reference, some Farnell codes: FET: 2453434 12V Zener: 1081407 6.2V Zener: 1081435"
- moved on the sheet: J8, Q8, Q9, R25, R64, R65, R66, R67, R68, R69, R70, R71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
