File: hardware/precharge/precharge.kicad_pcb (KiCad board)
At the start: 2 copper layers, 5 parts, among them K1 DIPxx-1Axx-13x, U1 OPAMP, U2 IL300, U3 OPAMP

Commit message: Assigned some footprints, created footprint library
Parts:
- added C1: 10u, Capacitor_SMD:C_0805_2012Metric, F.Cu at (106.7, 33.0)
- added C10: 100u, Capacitor_THT:CP_Radial_D8.0mm_P3.50mm, F.Cu at (42.6, 57.9)
- added C11: 100u, Capacitor_THT:CP_Radial_D8.0mm_P3.50mm, F.Cu at (52.3, 57.9)
- added C12: 100n, Capacitor_SMD:C_0603_1608Metric, F.Cu at (93.5, 39.8)
- added C13: 100u, Capacitor_THT:CP_Radial_D8.0mm_P3.50mm, F.Cu at (42.6, 67.5)
- added C2: 3.3u, Capacitor_SMD:C_0805_2012Metric, F.Cu at (101.8, 34.3)
- added C3: 22u, Capacitor_THT:CP_Radial_D8.0mm_P3.50mm, F.Cu at (62.0, 57.9)
- added C4: 4.7u, Capacitor_SMD:C_0805_2012Metric, F.Cu at (79.8, 23.6)
- added C5: 100n, Capacitor_SMD:C_0603_1608Metric, F.Cu at (61.2, 36.9)
- added C6: 22u, Capacitor_THT:CP_Radial_D8.0mm_P3.50mm, F.Cu at (52.3, 67.5)
- added C7: 100n, Capacitor_SMD:C_0603_1608Metric, F.Cu at (70.2, 29.1)
- added C8: 100n, Capacitor_SMD:C_0603_1608Metric, F.Cu at (65.3, 36.9)
- added C9: 100n, Capacitor_SMD:C_0603_1608Metric, F.Cu at (70.2, 31.6)
- added D1: SS14+, Diode_SMD:D_SMA, F.Cu at (32.1, 79.3)
- added D10: LED, LED_SMD:LED_0603_1608Metric, F.Cu at (42.2, 78.5)
- added D11: LED, LED_SMD:LED_0603_1608Metric, F.Cu at (46.3, 78.5)
- added D12: LED, LED_SMD:LED_0603_1608Metric, F.Cu at (57.6, 73.9)
- added D13: LED, LED_SMD:LED_0603_1608Metric, F.Cu at (89.5, 39.9)
- added D14: LED, LED_SMD:LED_0603_1608Metric, F.Cu at (75.1, 27.1)
- added D2: BAT54W, Package_TO_SOT_SMD:SOT-323_SC-70, F.Cu at (111.1, 24.7)
- added D3: BAT54W, Package_TO_SOT_SMD:SOT-323_SC-70, F.Cu at (106.7, 29.7)
- added D4: BAT54W, Package_TO_SOT_SMD:SOT-323_SC-70, F.Cu at (115.1, 20.3)
- added D5: BAT54W, Package_TO_SOT_SMD:SOT-323_SC-70, F.Cu at (119.6, 20.3)
- added D6: BAT54W, Package_TO_SOT_SMD:SOT-323_SC-70, F.Cu at (79.8, 20.3)
- added D7: BAT54W, Package_TO_SOT_SMD:SOT-323_SC-70, F.Cu at (75.3, 20.3)
- added D8: BAT54W, Package_TO_SOT_SMD:SOT-323_SC-70, F.Cu at (75.3, 23.9)
- added D9: LED, LED_SMD:LED_0603_1608Metric, F.Cu at (38.2, 78.5)
- added K2: G5Q-1, Relay_THT:Relay_SPDT_Omron-G5Q-1, F.Cu at (30.6, 28.5)
- added K3: G5Q-1, Relay_THT:Relay_SPDT_Omron-G5Q-1, F.Cu at (30.6, 41.1)
- added NT1: NetTie_2, NetTie:NetTie-2_SMD_Pad0.5mm, F.Cu at (97.0, 39.6)
- added NT2: NetTie_2, NetTie:NetTie-2_SMD_Pad0.5mm, F.Cu at (45.8, 49.0)
- added PS2: MPWF1212S-3W, Converter_DCDC:Converter_DCDC_XP_POWER-ITXxxxxSA_THT, F.Cu at (118.1, 54.5)
- added Q1: BC856, Package_TO_SOT_SMD:SOT-23, F.Cu at (106.4, 25.6)
- added Q2: BC856, Package_TO_SOT_SMD:SOT-23, F.Cu at (110.5, 20.7)
- added Q3: BC856, Package_TO_SOT_SMD:SOT-23, F.Cu at (102.0, 30.6)
- added Q6: XP262N7002TR-G, Package_TO_SOT_SMD:SOT-23, F.Cu at (65.7, 30.9)
- added Q7: XP262N7002TR-G, Package_TO_SOT_SMD:SOT-23, F.Cu at (46.7, 45.8)
- added Q8: XP262N7002TR-G, Package_TO_SOT_SMD:SOT-23, F.Cu at (70.6, 25.6)
- added R1: 1k, Resistor_SMD:R_0603_1608Metric, F.Cu at (41.4, 74.7)
- added R10: 680k, Resistor_SMD:R_0805_2012Metric, F.Cu at (111.1, 31.0)
- added R11: 33k, Resistor_SMD:R_0603_1608Metric, F.Cu at (89.4, 36.1)
- added R12: 680k, Resistor_SMD:R_0805_2012Metric, F.Cu at (115.5, 32.4)
- added R13: 680k, Resistor_SMD:R_0805_2012Metric, F.Cu at (110.6, 39.8)
- added R14: 680k, Resistor_SMD:R_0805_2012Metric, F.Cu at (110.6, 36.9)
- added R15: 680k, Resistor_SMD:R_0805_2012Metric, F.Cu at (119.9, 26.5)
- added R16: 33k, Resistor_SMD:R_0603_1608Metric, F.Cu at (97.5, 31.1)
- added R17: 120k, Resistor_SMD:R_0603_1608Metric, F.Cu at (97.5, 36.1)
- added R18: 1.5k, Resistor_SMD:R_0603_1608Metric, F.Cu at (101.9, 25.9)
- added R19: 30k, Resistor_SMD:R_0603_1608Metric, F.Cu at (93.5, 36.1)
- added R2: 1k, Resistor_SMD:R_0603_1608Metric, F.Cu at (53.5, 74.7)
- added R20: 680k, Resistor_SMD:R_0805_2012Metric, F.Cu at (115.0, 36.9)
- added R21: 680k, Resistor_SMD:R_0805_2012Metric, F.Cu at (119.9, 29.5)
- added R22: 680k, Resistor_SMD:R_0805_2012Metric, F.Cu at (106.2, 36.0)
- added R23: 560k, Resistor_SMD:R_0805_2012Metric, F.Cu at (111.1, 33.9)
- added R24: 100k, Resistor_SMD:R_0603_1608Metric, F.Cu at (97.9, 25.9)
- added R25: 680, Resistor_THT:R_Axial_Power_L75.0mm_W9.0mm_P86.36mm, F.Cu at (81.3, 81.3)
- added R26: 33k, Resistor_SMD:R_0603_1608Metric, F.Cu at (106.0, 20.9)
- added R27: 680k, Resistor_SMD:R_0805_2012Metric, F.Cu at (115.5, 29.5)
- added R28: 680k, Resistor_SMD:R_0805_2012Metric, F.Cu at (115.5, 23.6)
- added R29: 680k, Resistor_SMD:R_0805_2012Metric, F.Cu at (111.1, 28.0)
- added R3: 1k, Resistor_SMD:R_0603_1608Metric, F.Cu at (64.9, 65.2)
- added R30: 680k, Resistor_SMD:R_0805_2012Metric, F.Cu at (106.2, 39.0)
- added R31: 100k, Resistor_SMD:R_0603_1608Metric, F.Cu at (101.9, 20.9)
- added R32: 5.1M, Resistor_SMD:R_0603_1608Metric, F.Cu at (93.5, 31.1)
- added R35: 470k, Resistor_SMD:R_0603_1608Metric, F.Cu at (65.3, 34.4)
- added R36: 47k, Resistor_SMD:R_0603_1608Metric, F.Cu at (69.7, 20.9)
- added R37: 1k, Resistor_SMD:R_0603_1608Metric, F.Cu at (38.2, 46.0)
- added R38: 10k, Resistor_SMD:R_0603_1608Metric, F.Cu at (34.2, 46.0)
- added R39: 100k, Resistor_SMD:R_0603_1608Metric, F.Cu at (61.3, 31.1)
- added R4: 10k, Resistor_SMD:R_0603_1608Metric, F.Cu at (60.9, 70.1)
- added R40: 100k, Resistor_SMD:R_0603_1608Metric, F.Cu at (42.3, 46.0)
- added R41: 3.3k, Resistor_SMD:R_0603_1608Metric, F.Cu at (45.4, 74.7)
- added R42: 3.3k, Resistor_SMD:R_0603_1608Metric, F.Cu at (74.6, 55.6)
- added R43: 3.3k, Resistor_SMD:R_0603_1608Metric, F.Cu at (70.6, 55.6)
- added R44: 3.3k, Resistor_SMD:R_0603_1608Metric, F.Cu at (70.6, 60.6)
- added R45: 3.3k, Resistor_SMD:R_0603_1608Metric, F.Cu at (97.9, 20.9)
- added R46: 3.3k, Resistor_SMD:R_0603_1608Metric, F.Cu at (30.1, 46.0)
- added R5: 10k, Resistor_SMD:R_0603_1608Metric, F.Cu at (49.5, 74.7)
- added R6: 10k, Resistor_SMD:R_0603_1608Metric, F.Cu at (60.9, 65.2)
- added R7: 680k, Resistor_SMD:R_0805_2012Metric, F.Cu at (115.5, 26.5)
- added R8: 680k, Resistor_SMD:R_0805_2012Metric, F.Cu at (101.8, 37.3)
- added R9: 680k, Resistor_SMD:R_0805_2012Metric, F.Cu at (119.9, 23.6)
- added TH1: NCU18WF104J60RB, Resistor_SMD:R_0603_1608Metric, F.Cu at (61.2, 39.4)
- added U4: TLV274, Package_SO:SOIC-14_3.9x8.7mm_P1.27mm, F.Cu at (91.6, 23.6)
- added U5: 40106, Package_SO:SOIC-14_3.9x8.7mm_P1.27mm, F.Cu at (55.0, 33.8)
- added U6: LM339, Package_SO:SOIC-14_3.9x8.7mm_P1.27mm, F.Cu at (63.5, 23.6)
- added U7: 4013, Package_SO:SOIC-14_3.9x8.7mm_P1.27mm, F.Cu at (55.0, 44.0)
- added U8: 4001, Package_SO:SOIC-14_3.9x8.7mm_P1.27mm, F.Cu at (55.0, 23.6)
- K1: value DIPxx-1Axx-13x -> DIPxx-1Cxx-51x
- PS1: value IA1212D -> MPWF1212S-3W; footprint Converter_DCDC:Converter_DCDC_XP_POWER-IAxxxxD_THT -> Converter_DCDC:Converter_DCDC_XP_POWER-ITXxxxxSA_THT
- U1, U3: value OPAMP -> 140817141410; footprint Package_TO_SOT_SMD:SOT-23-5 -> Package_DIP:DIP-4_W7.62mm
- U2: value IL300 -> 140817141410; footprint Package_DIP:DIP-8_W7.62mm -> Package_DIP:DIP-4_W7.62mm
- moved PS1 4.20 mm to (118.1, 39.2)
Connections:
- K1 pad 1: (no net) -> Net-(K1-Pad1)
- K1 pad 14: unconnected-(K1-Pad14) -> Net-(J2-Pad1)
- K1 pad 2: unconnected-(K1-Pad2) -> /LV side/RELAY-
- K1 pad 6: Net-(K1-Pad6) -> /LV side/RELAY+
- K1 pad 7: (no net) -> /HV side/HV_IN
- K1 pad 8: Net-(K1-Pad8) -> /HV side/HV_IN
- PS1 pad 1: Net-(K1-Pad6) -> GND
- PS1 pad 2: unconnected-(PS1-Pad2) -> +12V
- U1 pad 1: unconnected-(U1-Pad1) -> Net-(R1-Pad2)
- U1 pad 2: Net-(R1-Pad1) -> Net-(K1-Pad1)
- U1 pad 3: Net-(R2-Pad1) -> /~{PRECHARGE_RELAY_ON}
- U1 pad 4: Net-(PS1-Pad5) -> +12V
- U2 pad 2: Net-(PS1-Pad6) -> /HV side/~{CHARGED}
- U2 pad 3: Net-(PS1-Pad5) -> /LV side/CHARGED
- U2 pad 4: Net-(R1-Pad1) -> +12V
- U3 pad 1: Net-(R3-Pad2) -> /HV side/~{TIMING_FAULT_OC}
- U3 pad 2: Net-(U3-Pad2) -> /HV side/GND
- U3 pad 3: Net-(U3-Pad2) -> /LV side/~{TIMING_FAULT}
- U3 pad 4: Net-(R3-Pad1) -> +12V

Commit message: Preliminary PCB placement
Parts:
- added F1: Fuse, footprints:fuseholder, F.Cu at (141.0, 44.8)
- added J1: Conn_01x02, Connector_PinHeader_2.54mm:PinHeader_1x02_P2.54mm_Horizontal, F.Cu at (50.4, 25.7)
- added J2: Conn_01x01, Connector_PinHeader_2.54mm:PinHeader_1x01_P2.54mm_Horizontal, F.Cu at (63.8, 21.1)
- added J3: Conn_01x05, Connector_PinHeader_2.54mm:PinHeader_1x05_P2.54mm_Horizontal, F.Cu at (209.6, 92.7)
- added J4: Conn_01x04, Connector_PinHeader_2.54mm:PinHeader_1x04_P2.54mm_Horizontal, F.Cu at (209.6, 52.1)
- added J5: Conn_01x01, Connector_PinHeader_2.54mm:PinHeader_1x01_P2.54mm_Horizontal, F.Cu at (50.4, 21.1)
- C1: value 10u -> 100u; footprint Capacitor_SMD:C_0805_2012Metric -> Capacitor_THT:CP_Radial_D6.3mm_P2.50mm
- C10, C11: footprint Capacitor_THT:CP_Radial_D8.0mm_P3.50mm -> Capacitor_THT:CP_Radial_D6.3mm_P2.50mm
- C13: value 100u -> 4.7u; footprint Capacitor_THT:CP_Radial_D8.0mm_P3.50mm -> Capacitor_THT:CP_Radial_D5.0mm_P2.00mm
- C2: value 3.3u -> 10u; footprint Capacitor_SMD:C_0805_2012Metric -> Capacitor_THT:CP_Radial_D5.0mm_P2.00mm
- C4: value 4.7u -> 3.3u; footprint Capacitor_SMD:C_0805_2012Metric -> Capacitor_THT:CP_Radial_D5.0mm_P2.00mm
- K2, K3: value G5Q-1 -> G5Q-1EU DC12
- PS2: footprint Converter_DCDC:Converter_DCDC_XP_POWER-ITXxxxxSA_THT -> footprints:MPWF1212S-3W
- R25: footprint Resistor_THT:R_Axial_Power_L75.0mm_W9.0mm_P86.36mm -> footprints:HSA50680RJ
- moved U1 210.0 mm to (-34.3, 25.4)
- moved K1 190.9 mm to (-39.4, 1.29)
- moved D9 182.6 mm to (217.2, 42.5)
- moved D1 174.9 mm to (207.0, 80.6), turned to -90 degrees
- moved R41 174.0 mm to (215.9, 40.0)
- moved R38 168.1 mm to (194.9, 95.2)
- moved NT2 167.7 mm to (213.4, 42.5)
- moved D10 167.3 mm to (208.9, 63.5), turned to 180 degrees
- moved R37 167.1 mm to (195.6, 102.2), turned to -90 degrees
- moved R46 163.1 mm to (186.1, 94.0)
- moved D11 163.0 mm to (208.9, 67.9), turned to 180 degrees
- moved R40 160.1 mm to (196.8, 87.6)
- moved U6 157.5 mm to (201.3, 99.7)
- moved K3 156.7 mm to (186.1, 60.3)
- moved K2 156.7 mm to (186.1, 47.6)
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Connections:
- C1 pad 1: Net-(C1-Pad1) -> +12V
- C1 pad 2: /HV side/GND -> GND
- C13 pad 1: +12V -> Net-(R40-Pad1)
- C2 pad 1: Net-(C2-Pad1) -> Net-(R10-Pad1)
- C4 pad 1: GND -> Net-(Q1-Pad1)
- C4 pad 2: Net-(C4-Pad2) -> /HV side/GND
- Q1 pad 1: Net-(C2-Pad1) -> Net-(Q1-Pad1)
- R10 pad 1: Net-(C1-Pad1) -> Net-(R10-Pad1)
- R11 pad 1: Net-(C1-Pad1) -> Net-(R10-Pad1)
- R15 pad 1: Net-(C2-Pad1) -> Net-(Q1-Pad1)
- R16 pad 1: Net-(C2-Pad1) -> Net-(Q1-Pad1)
- R40 pad 1: Net-(C4-Pad2) -> Net-(R40-Pad1)
- U4 pad 9: Net-(C1-Pad1) -> Net-(R10-Pad1)
- U5 pad 9: Net-(C4-Pad2) -> Net-(R40-Pad1)
Other:
- board outline added: 111.8 x 81.3 mm

Commit message: Added support for TS_ACTIVE signal, adjusted resistor divider
Parts:
- removed C11: 100u, Capacitor_THT:CP_Radial_D6.3mm_P2.50mm
- removed C5: 100n, Capacitor_SMD:C_0603_1608Metric
- removed K1: DIPxx-1Cxx-51x, Relay_THT:Relay_StandexMeder_DIP_LowProfile
- removed PS1: MPWF1212S-3W, Converter_DCDC:Converter_DCDC_XP_POWER-ITXxxxxSA_THT
- removed U6: LM339, Package_SO:SOIC-14_3.9x8.7mm_P1.27mm
- added D15: BAT54W, Package_TO_SOT_SMD:SOT-323_SC-70, F.Cu at (211.4, 21.3)
- added D16: BAT54W, Package_TO_SOT_SMD:SOT-323_SC-70, F.Cu at (211.4, 17.7)
- added J6: Conn_01x06, Connector_PinHeader_2.54mm:PinHeader_1x06_P2.54mm_Horizontal, F.Cu at (229.9, 66.0)
- added Q4: BC846, Package_TO_SOT_SMD:SOT-23, F.Cu at (203.2, 28.3)
- added R33: 1k, Resistor_SMD:R_0603_1608Metric, F.Cu at (185.8, 17.1)
- added R34: 1k, Resistor_SMD:R_0603_1608Metric, F.Cu at (189.8, 19.6)
- added R47: 1.5k, Resistor_SMD:R_0603_1608Metric, F.Cu at (189.8, 17.1)
- added R48: 1.5k, Resistor_SMD:R_0603_1608Metric, F.Cu at (185.8, 19.6)
- added R49: 1.5k, Resistor_SMD:R_0603_1608Metric, F.Cu at (198.1, 21.6)
- added R50: 1.5k, Resistor_SMD:R_0603_1608Metric, F.Cu at (193.8, 17.1)
- added R51: 470k, Resistor_SMD:R_0603_1608Metric, F.Cu at (137.0, 27.3)
- added R52: 47k, Resistor_SMD:R_0603_1608Metric, F.Cu at (141.0, 24.8)
- added R53: 1k, Resistor_SMD:R_0603_1608Metric, F.Cu at (137.0, 24.8)
- added R54: 10k, Resistor_SMD:R_0603_1608Metric, F.Cu at (207.6, 27.3)
- added U9: 4013, Package_SO:SOIC-14_3.9x8.7mm_P1.27mm, F.Cu at (201.3, 105.4)
- C6: value 22u -> 100n; footprint Capacitor_THT:CP_Radial_D8.0mm_P3.50mm -> Capacitor_SMD:C_0603_1608Metric
- J3: value Conn_01x05 -> Conn_01x02; footprint Connector_PinHeader_2.54mm:PinHeader_1x05_P2.54mm_Horizontal -> Connector_PinHeader_2.54mm:PinHeader_1x02_P2.54mm_Horizontal
- J5: value Conn_01x01 -> Conn_01x03; footprint Connector_PinHeader_2.54mm:PinHeader_1x01_P2.54mm_Horizontal -> Connector_PinHeader_2.54mm:PinHeader_1x03_P2.54mm_Horizontal
- R1, R2, R3: footprint Resistor_SMD:R_0603_1608Metric -> Resistor_SMD:R_1206_3216Metric
- R35: value 470k -> 1k
- R36: value 47k -> 1k
- R38: value 10k -> 1.5k
- U8: value 4001 -> 4071
- moved C6 239.8 mm to (200.5, 99.1)
- moved R4 228.6 mm to (177.8, 81.3)
- moved U1 211.2 mm to (168.3, 85.1)
- moved R1 191.2 mm to (162.6, 85.1)
- moved J5 179.9 mm to (210.9, 102.2)
- moved J1 125.9 mm to (144.1, 109.8), turned to 90 degrees
- moved J2 107.1 mm to (142.3, 94.0)
- moved TH1 71.8 mm to (125.7, 75.6)
- moved R36 39.4 mm to (234.9, 96.5)
- moved R37 39.4 mm to (234.9, 100.3)
- moved R35 39.2 mm to (231.1, 92.7)
- moved C10 10.2 mm to (179.2, 106.7)
- moved C3 10.2 mm to (167.4, 108.0)
- moved PS2 10.2 mm to (179.7, 99.1)
- moved NT1 10.00 mm to (150.5, 113.0)
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Connections:
- C10 pad 2: GND -> /LV side/GND
- C12 pad 1: /HV side/+12V -> /HV_+12V
- C12 pad 2: /HV side/GND -> /HV_GND
- C13 pad 2: GND -> /LV side/GND
- C2 pad 2: /HV side/GND -> /HV_GND
- C3 pad 1: /HV side/+12V -> /HV_+12V
- C3 pad 2: /HV side/GND -> /HV_GND
- C4 pad 2: /HV side/GND -> /HV_GND
- C6 pad 1: Net-(C6-Pad1) -> +12V
- C6 pad 2: /HV side/HV_IN -> /LV side/GND
- C7 pad 2: GND -> /LV side/GND
- C8 pad 2: GND -> /LV side/GND
- C9 pad 2: GND -> /LV side/GND
- D13 pad 2: /HV side/+12V -> /HV_+12V
- D2 pad 1: /HV side/+12V -> /HV_+12V
- D8 pad 1: /LV side/RELAY- -> /RELAY-
- J2 pad 1: Net-(J2-Pad1) -> /HV side/HV_IN
- J3 pad 1: /LV side/OVERTEMP_FAULT -> /RELAY-
- J3 pad 2: /LV side/TIMING_FAULT_OUT -> /LV side/RELAY+
- J5 pad 1: /~{PRECHARGE_RELAY_ON} -> /RELAY-
- NT1 pad 1: /HV side/GND -> /HV_GND
- PS2 pad 1: GND -> /LV side/GND
- PS2 pad 6: /HV side/+12V -> /HV_+12V
- PS2 pad 7: /HV side/GND -> /HV_GND
- Q1 pad 3: /HV side/GND -> /HV_GND
- Q2 pad 3: /HV side/GND -> /HV_GND
- Q3 pad 3: /HV side/GND -> /HV_GND
- Q6 pad 2: GND -> /LV side/GND
- Q7 pad 2: GND -> /LV side/GND
- Q8 pad 2: GND -> /LV side/GND
- Q8 pad 3: /LV side/RELAY- -> /RELAY-
- R1 pad 1: Net-(C6-Pad1) -> Net-(R1-Pad1)
- R1 pad 2: Net-(R1-Pad2) -> /HV_+12V
- R11 pad 2: /HV side/GND -> /HV_GND
- R16 pad 2: /HV side/GND -> /HV_GND
- R19 pad 2: /HV side/GND -> /HV_GND
- R2 pad 1: /HV side/+12V -> /HV_+12V
- R24 pad 1: /HV side/+12V -> /HV_+12V
- R26 pad 2: /HV side/GND -> /HV_GND
- R3 pad 2: /HV side/+12V -> /HV_+12V
- R31 pad 1: /HV side/+12V -> /HV_+12V
- R35 pad 1: +12V -> /LV side/FAULT
- R35 pad 2: Net-(R35-Pad2) -> Net-(J6-Pad3)
- R36 pad 1: +12V -> /LV side/PRECHARGE_ENABLED
- R36 pad 2: Net-(R36-Pad2) -> Net-(J6-Pad4)
- R37 pad 1: Net-(R36-Pad2) -> /LV side/AWAKE
- R37 pad 2: GND -> Net-(J6-Pad5)
- R38 pad 1: +12V -> GND
- R38 pad 2: Net-(R38-Pad2) -> Net-(J6-Pad1)
- R39 pad 2: GND -> /LV side/GND
- R4 pad 1: /~{PRECHARGE_RELAY_ON} -> +12V
- R4 pad 2: GND -> /LV side/OVERTEMP_FAULT
- R41 pad 2: /LV side/RELAY- -> /RELAY-
- R45 pad 2: /HV side/GND -> /HV_GND
- R46 pad 2: GND -> /LV side/GND
- TH1 pad 1: Net-(R35-Pad2) -> Net-(U4-Pad13)
- TH1 pad 2: GND -> /HV_GND
- U1 pad 1: Net-(R1-Pad2) -> Net-(R1-Pad1)
- U1 pad 2: Net-(K1-Pad1) -> /HV side/OVERTEMP_FAULT
- U1 pad 3: /~{PRECHARGE_RELAY_ON} -> GND
- U1 pad 4: +12V -> /LV side/OVERTEMP_FAULT
- U3 pad 2: /HV side/GND -> /HV_GND
- U4 pad 11: /HV side/GND -> /HV_GND
- U4 pad 12: /HV side/+12V -> Net-(U4-Pad12)
- U4 pad 13: /HV side/GND -> Net-(U4-Pad13)
- U4 pad 14: unconnected-(U4-Pad14) -> /HV side/OVERTEMP_FAULT
- U4 pad 4: /HV side/+12V -> /HV_+12V
- U5 pad 12: /LV side/FAULT -> Net-(Q6-Pad1)
- U5 pad 7: GND -> /LV side/GND
- U7 pad 1: /LV side/OVERTEMP_FAULT -> /LV side/OVERTEMP_FAULT_OUT
- U7 pad 11: GND -> /LV side/GND
- U7 pad 3: GND -> /LV side/GND
- U7 pad 5: GND -> /LV side/GND
- U7 pad 6: Net-(R38-Pad2) -> /LV side/OVERTEMP_FAULT
- U7 pad 7: GND -> /LV side/GND
- U7 pad 9: GND -> /LV side/GND
- U8 pad 1: /LV side/TIMING_FAULT_OUT -> /LV side/FAULT
- U8 pad 12: GND -> /LV side/GND
- U8 pad 13: GND -> /LV side/GND
- U8 pad 2: /LV side/OVERTEMP_FAULT -> /LV side/~{TS_ENABLED}
- U8 pad 4: Net-(Q6-Pad1) -> /LV side/FAULT
- U8 pad 5: /LV side/FAULT -> /LV side/TIMING_FAULT_OUT
- U8 pad 6: /LV side/POR -> /LV side/OVERTEMP_FAULT_OUT
- U8 pad 7: GND -> /LV side/GND
- U8 pad 8: GND -> /LV side/GND
- U8 pad 9: GND -> /LV side/GND
